Commit message: start MPC

File: legged_controllers/config/h1/h1_cbf.urdf (robot description, URDF)
Before this commit: robot h1_description, 29 links, 28 joints
Links:
- removed link leg_l_f1_link
- removed link leg_l_f2_link
- removed link leg_r_f1_link
- removed link leg_r_f2_link
Joints:
- removed joint leg_l5_fixed_1
- removed joint leg_l5_fixed_2
- removed joint leg_r5_fixed_1
- removed joint leg_r5_fixed_2
