Commit message: finish interface and dummy

File: h1_description/urdf/h1_cbf_control.urdf (robot description, URDF)
Before this commit: robot h1_description, 29 links, 28 joints
Links:
- removed link leg_l_f1_link
- removed link leg_l_f2_link
- removed link leg_r_f1_link
- removed link leg_r_f2_link
- link d435_left_imager_link: geometry collision sphere radius=0.001
- link d435_rgb_module_link: geometry collision sphere radius=0.001
- link imu_link: geometry 
- link left_ankle_link: geometry collision box size=0.28 0.03 0.024
- link left_elbow_link: geometry collision cylinder length=0.09 radius=0.03
- link left_hip_pitch_link: geometry collision cylinder length=0.2 radius=0.05
- link left_hip_roll_link: geometry collision cylinder length=0.01 radius=0.02
- link left_hip_yaw_link: geometry collision cylinder length=0.02 radius=0.01
- link left_knee_link: geometry collision cylinder length=0.2 radius=0.05
- link left_shoulder_pitch_link: geometry collision cylinder length=0.04 radius=0.03
- link left_shoulder_roll_link: geometry collision cylinder length=0.01 radius=0.04
- link left_shoulder_yaw_link: geometry collision cylinder length=0.01 radius=0.04
- link logo_link: geometry 
- link mid360_link: geometry collision sphere radius=0.001
- link pelvis: geometry collision sphere radius=0.05
- link right_ankle_link: geometry collision box size=0.28 0.03 0.024
- link right_elbow_link: geometry collision cylinder length=0.09 radius=0.03
- link right_hip_pitch_link: geometry collision cylinder length=0.2 radius=0.05
- link right_hip_roll_link: geometry collision cylinder length=0.01 radius=0.02
- link right_hip_yaw_link: geometry collision cylinder length=0.02 radius=0.01
- link right_knee_link: geometry collision cylinder length=0.2 radius=0.05
- link right_shoulder_pitch_link: geometry collision cylinder length=0.04 radius=0.03
- link right_shoulder_roll_link: geometry collision cylinder length=0.01 radius=0.04
- link right_shoulder_yaw_link: geometry collision cylinder length=0.01 radius=0.04
- link torso_link: geometry collision box size=0.08 0.16 0.1
Joints:
- removed joint leg_l5_fixed_1
- removed joint leg_l5_fixed_2
- removed joint leg_r5_fixed_1
- removed joint leg_r5_fixed_2
- joint left_elbow_joint: type fixed -> revolute
- joint left_shoulder_pitch_joint: type fixed -> revolute
- joint left_shoulder_roll_joint: type fixed -> revolute
- joint left_shoulder_yaw_joint: type fixed -> revolute
- joint right_elbow_joint: type fixed -> revolute
- joint right_shoulder_pitch_joint: type fixed -> revolute
- joint right_shoulder_roll_joint: type fixed -> revolute
- joint right_shoulder_yaw_joint: type fixed -> revolute
- joint torso_joint: type fixed -> revolute
