Commit message: update

File: h1_description/urdf/h1_dynamic.urdf (robot description, URDF)
Before this commit: robot h1_description, 29 links, 28 joints
Links:
- link leg_l_f1_link: geometry collision sphere radius=0.01; visual sphere radius=0.01
- link leg_l_f2_link: geometry collision sphere radius=0.01; visual sphere radius=0.01
- link leg_r_f1_link: geometry collision sphere radius=0.01; visual sphere radius=0.01
- link leg_r_f2_link: geometry collision sphere radius=0.01; visual sphere radius=0.01
Joints:
- joint leg_l5_fixed_1: origin xyz=0.2 0 -0.03 rpy=0 0 0 -> xyz=0.2 0 -0.065 rpy=0 0 0
- joint leg_l5_fixed_2: origin xyz=-0.1 0 -0.03 rpy=0 0 0 -> xyz=-0.1 0 -0.065 rpy=0 0 0
- joint leg_r5_fixed_1: origin xyz=0.2 0 -0.03 rpy=0 0 0 -> xyz=0.2 0 -0.065 rpy=0 0 0
- joint leg_r5_fixed_2: origin xyz=-0.1 0 -0.03 rpy=0 0 0 -> xyz=-0.1 0 -0.065 rpy=0 0 0

Commit message: finish wbc and simulation

File: h1_description/urdf/h1_dynamic.urdf (robot description, URDF)
Before this commit: robot h1_description, 29 links, 28 joints
Joints:
- joint leg_l5_fixed_1: origin xyz=0.2 0 -0.065 rpy=0 0 0 -> xyz=0.2 0 -0.06 rpy=0 0 0
- joint leg_l5_fixed_2: origin xyz=-0.1 0 -0.065 rpy=0 0 0 -> xyz=-0.1 0 -0.06 rpy=0 0 0
- joint leg_r5_fixed_1: origin xyz=0.2 0 -0.065 rpy=0 0 0 -> xyz=0.2 0 -0.06 rpy=0 0 0
- joint leg_r5_fixed_2: origin xyz=-0.1 0 -0.065 rpy=0 0 0 -> xyz=-0.1 0 -0.06 rpy=0 0 0
