Commit message: update

File: h1_description/urdf/h1_dynamic_old.urdf (robot description, URDF)
Before this commit: robot h1_description, 30 links, 29 joints
Links:
- removed link base
Joints:
- removed joint pelvis_joint
- joint imu_joint: origin xyz=0 0 0 rpy=0 0 0 -> xyz=-0.04452 -0.01891 0.27756 rpy=0 0 0; parent base -> torso_link
